Commit message: Fixed up xacros

File: urdf/sensors.urdf.xacro (robot description, xacro)
@@ -7,5 +7,5 @@
   <!-- Front LiDAR  -->
   <xacro:include filename="$(find my_package)/urdf/sick_lms1xx_mount.urdf.xacro" />
-  <sick_lms1xx_mount prefix="$(optenv JACKAL_LASER_MOUNT front)"
+  <xacro:sick_lms1xx_mount prefix="$(optenv JACKAL_LASER_MOUNT front)"
                      topic="$(optenv JACKAL_LASER_TOPIC /front_lidar_scan)"/>
   <joint name="$(optenv JACKAL_LASER_MOUNT front)_laser_mount_joint" type="fixed">
@@ -16,6 +16,7 @@
   </joint>
   <!-- Rear LiDAR  -->
-  <xacro:include filename="$(find my_package)/urdf/sick_lms1xx_mount.urdf.xacro" />
-  <sick_lms1xx_mount prefix="$(optenv JACKAL_LASER_MOUNT rear)"
+  <!-- Removed.  Included above already -->
+  <!-- xacro:include filename="$(find my_package)/urdf/sick_lms1xx_mount.urdf.xacro" / -->
+  <xacro:sick_lms1xx_mount prefix="$(optenv JACKAL_LASER_MOUNT rear)"
                      topic="$(optenv JACKAL_LASER_TOPIC /rear_lidar_scan)"/>
   <joint name="$(optenv JACKAL_LASER_MOUNT rear)_laser_mount_joint" type="fixed">

File: urdf/sick_lms1xx_mount.urdf.xacro (robot description, xacro)
@@ -45,4 +45,6 @@
       <child link="${prefix}_laser" />
     </joint>
+    <!-- This link didn't exis, but it is listed as the child of the joint above -->
+    <link name="${prefix}_laser" />
     <gazebo reference="${prefix}_laser_mount">
       <material>Gazebo/DarkGrey</material>
